File: passive-ethernet-tap/passive-ethernet-tap.kicad_pcb (KiCad board)
At the start: 2 copper layers, 82 x 40.9 mm, 4 parts, among them J1 Device_A, J2 Sniff_A, J3 Sniff_B, J4 Device_B

Commit message: Apparently mounting holes dissapeared
Parts:
- added REF**: MountingHole_3mm, MountingHole:MountingHole_3mm, F.Cu at (110.0, 54.0)
- added REF**: MountingHole_3mm, MountingHole:MountingHole_3mm, F.Cu at (156.8, 54.1)
- added REF**: MountingHole_3mm, MountingHole:MountingHole_3mm, F.Cu at (133.3, 35.2)
Changed lines of the file:
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@@
     )
+  )
+  (footprint "MountingHole:MountingHole_3mm" (layer "F.Cu")
+    (at 109.982 53.975)
+    (descr "Mounting Hole 3mm, no annular")
+    (tags "mounting hole 3mm no annular")
+    (attr exclude_from_pos_files exclude_from_bom)
+    (fp_text reference "REF**" (at 0 -4) (layer "F.SilkS") hide
+      (effects (font (size 1 1) (thickness 0.15)))
+    )
+    (fp_text value "MountingHole_3mm" (at 0 4) (layer "F.Fab")
+      (effects (font (size 1 1) (thickness 0.15)))
+    )
+    (fp_text user "${REFERENCE}" (at 0 0) (layer "F.Fab")
+      (effects (font (size 1 1) (thickness 0.15)))
+    )
+    (fp_circle (center 0 0) (end 3 0) (layer "Cmts.User") (width 0.15) (fill none))
+    (fp_circle (center 0 0) (end 3.25 0) (layer "F.CrtYd") (width 0.05) (fill none))
+    (pad "" np_thru_hole circle (at 0 0) (size 3 3) (drill 3) (layers *.Cu *.Mask))
   )
   (footprint "ProjectSpecificParts:Bel Fuse SS-90000-011" (layer "F.Cu")
@@
       (rotate (xyz -90 0 0))
     )
+  )
+  (footprint "MountingHole:MountingHole_3mm" (layer "F.Cu")
+    (at 156.845 54.102)
+    (descr "Mounting Hole 3mm, no annular")
+    (tags "mounting hole 3mm no annular")
+    (attr exclude_from_pos_files exclude_from_bom)
+    (fp_text reference "REF**" (at 0 -4) (layer "F.SilkS") hide
+      (effects (font (size 1 1) (thickness 0.15)))
+    )
+    (fp_text value "MountingHole_3mm" (at 0 4) (layer "F.Fab")
+      (effects (font (size 1 1) (thickness 0.15)))
+    )
+    (fp_text user "${REFERENCE}" (at 0 0) (layer "F.Fab")
+      (effects (font (size 1 1) (thickness 0.15)))
+    )
+    (fp_circle (center 0 0) (end 3 0) (layer "Cmts.User") (width 0.15) (fill none))
+    (fp_circle (center 0 0) (end 3.25 0) (layer "F.CrtYd") (width 0.05) (fill none))
+    (pad "" np_thru_hole circle (at 0 0) (size 3 3) (drill 3) (layers F&B.Cu *.Mask))
   )
   (footprint "ProjectSpecificParts:Bel Fuse SS-90000-011" (layer "F.Cu")
@@
     )
   )
+  (footprint "MountingHole:MountingHole_3mm" (layer "F.Cu")
+    (at 133.35 35.179)
+    (descr "Mounting Hole 3mm, no annular")
+    (tags "mounting hole 3mm no annular")
+    (attr exclude_from_pos_files exclude_from_bom)
+    (fp_text reference "REF**" (at 0 -4) (layer "F.SilkS") hide
+      (effects (font (size 1 1) (thickness 0.15)))
+    )
+    (fp_text value "MountingHole_3mm" (at 0 4) (layer "F.Fab")
+      (effects (font (size 1 1) (thickness 0.15)))
+    )
+    (fp_text user "${REFERENCE}" (at 0 0) (layer "F.Fab")
+      (effects (font (size 1 1) (thickness 0.15)))
+    )
+    (fp_circle (center 0 0) (end 3 0) (layer "Cmts.User") (width 0.15) (fill none))
+    (fp_circle (center 0 0) (end 3.25 0) (layer "F.CrtYd") (width 0.05) (fill none))
+    (pad "" np_thru_hole circle (at 0 0) (size 3 3) (drill 3) (layers F&B.Cu *.Mask))
+  )
   (gr_line (start 92.329 30.607) (end 92.329 49.657) (layer "Edge.Cuts") (width 0.1))
